File: pcb/kicad/antenna/patch.kicad_pcb (KiCad board)
At the start: 2 copper layers, 1 part, among them P1 CONN_01X02

Commit message: Add pdf and archive of initial design
Other:
- board text added: "0.1"
- board text added: "February 15, 2017"
- board text added: "Patch Test Board"
Changed lines of the file:
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@@
     (links 9)
     (no_connects 4)
-    (area 0 0 0 0)
+    (area 111.76 54.61 158.750001 136.435001)
     (thickness 1.5748)
-    (drawings 0)
+    (drawings 3)
     (tracks 0)
     (zones 0)
@@
     (40 Dwgs.User user)
     (41 Cmts.User user)
-    (42 Eco1.User user)
-    (43 Eco2.User user)
+    (42 Eco1.User user hide)
+    (43 Eco2.User user hide)
     (44 Edge.Cuts user)
     (45 Margin user)
@@
   )
   (setup
-    (last_trace_width 2.54)
+    (last_trace_width 0.25)
     (user_trace_width 0.3556)
     (user_trace_width 2.54)
@@
     (pad_to_mask_clearance 0.2)
     (aux_axis_origin 12.065 12.065)
+    (grid_origin 127.635 85.725)
     (visible_elements 7FFFFFFF)
     (pcbplotparams
@@
       (net 2 GND))
   )
+  (gr_text "February 15, 2017" (at 217.17 193.04) (layer Cmts.User)
+    (effects (font (size 1.5 1.5) (thickness 0.3)))
+  )
+  (gr_text 0.1 (at 270.51 193.04) (layer Cmts.User)
+    (effects (font (size 1.5 1.5) (thickness 0.3)))
+  )
+  (gr_text "Patch Test Board" (at 196.215 189.23) (layer Cmts.User)
+    (effects (font (size 1.5 1.5) (thickness 0.3)))
+  )
   (zone (net 2) (net_name GND) (layer B.Cu) (hatch full 0.508)
