File: pcb/kicad/base/base.sch (KiCad schematic (older format))
At the start: 0 parts

Commit message: Add initial schematic for base central
Added the crystal and antenna circuitry with a combinations of reference
and placeholder values. SWD debugger connection is partially complete.
Parts:
- added AE1: 2.4-2.4835GHz, symbol Antenna
- added C1, C2, C3, C4, C8, C9: C_Small, symbol C_Small
- added C5: 3.9pF, symbol C_Small
- added C6: DNI, symbol C_Small
- added C7: 1.1pF, symbol C_Small
- added L1: 4.3nH, symbol L_Small
- added L2: L_Small, symbol L_Small
- added P1: CONN_01X02, symbol CONN_01X02
- added P?: CONN_02X10, symbol CONN_02X10
- added U1: SAMB11G18A, QFN-48-1EP_6x6mm_Pitch0.4mm, symbol SAMB11G18A
- added Y1: 26MHz, symbol Crystal_GND3_Small
- added Y2: 32.768kHz, symbol Crystal_GND3_Small
Connections:
- net labels added: GND, SWCLK, SWDIO
- wire segments 0 -> 33
- no-connect marks 0 -> 5
Other:
- note added: "1.0"
- note added: "Base - Central"
- note added: "March 2, 2017"
