File: pcb/button_1_0/button_1_00.sch (KiCad schematic (older format))
At the start: 71 parts, among them J1 JTAG_10x2, J10 GND_OUT, J11 PWR_OUT, J12 GPIO0/1_O, J13 GPIO9/10, J14 IO_BOT, J15 IO_BOT_O, J16 GPIO0/1, J17 RESET, J2 IO_UP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

Commit message: recommit_4_9
Parts:
- U1: footprint uCs:QFN-32-1EP_5x5mm -> uCs:STBNRG1
Changed lines of the file:
@@
 F 0 "U1" H 7850 2150 50  0000 C CNN
 F 1 "STBlueNRG-1" H 7050 3100 50  0000 C CNN
-F 2 "uCs:QFN-32-1EP_5x5mm" H 7700 2000 50  0001 C CIN
+F 2 "uCs:STBNRG1" H 7700 2000 50  0001 C CIN
 F 3 "" H 7000 2850 50  0001 C CNN
 	1    7000 2850
