File: pcb/kicad/button/button_mkii/button.sch (KiCad schematic (older format))
At the start: 42 parts, among them J1 SWD with less, U1 STBlueNRG-1, Y1 Xtal 32.768kHz, Y2 XTAL 16MHz

Commit message: updated design, layout, and appnotes; rev3
Parts:
- removed D1: Power thru SWD, Diodes_SMD:D_0603, symbol D_Schottky
- removed L2, L3: RFC, Miscellaneous:L_0402, symbol L
- added C20, C21: 1uF, Capacitors_SMD:C_0402, symbol C
- added C22: 1uF, Capacitors_SMD:C_0805, symbol C
- added C23: 0.1uF, Capacitors_SMD:C_0603, symbol C
- added C24: 0.01uF, Capacitors_SMD:C_0402, symbol C
- added R16: 1k, Resistors_SMD:R_0402, symbol R
- added TP7: Xtal32MHz, Miscellaneous:Measurement_Point_Round-SMD-tiniest, symbol TEST
- added TP8: Xtal32kHz, Miscellaneous:Measurement_Point_Round-SMD-tiniest, symbol TEST
- added U2: TLV1117LV-3V, TO_SOT_Packages_SMD:SOT-223, symbol LT1129CST-3.3
- C1: value 100pF -> 1uF; footprint Capacitors_SMD:C_0402 -> Capacitors_SMD:C_0805
- C14: value 22pF -> 27pF
- C15: value 18pF -> 33pF
- C2: footprint Capacitors_SMD:C_0402 -> Capacitors_SMD:C_0603
- C3: value 2.2pF -> 0.01uF
- C4: value 1000pF -> 0.01uF; footprint Capacitors_SMD:C_0402 -> Capacitors_SMD:C_0805
- C5: value 2.2uF -> 1000pF; footprint Capacitors_SMD:C_0402 -> Capacitors_SMD:C_0603
- C7: value 10pF -> 0.01uF; footprint Capacitors_SMD:C_0402 -> Capacitors_SMD:C_0805
- C8: value 1uF -> 1000pF; footprint Capacitors_SMD:C_0402 -> Capacitors_SMD:C_0603
- C9: value 1000pF -> 10pF
- R6: value 100k -> 1k; footprint Resistors_SMD:R_0603 -> Resistors_SMD:R_0402
- Y2: value XTAL 16MHz -> XTAL 32MHz
Connections:
- net +3V3: now also C4.1, C5.1, C6.1, J1.6 (P6), R4.1, R8.2, C21.2, C22.2, C23.2, C24.2, U2.2 (OUT); no longer C4.2, C5.2, C6.2, J1.1 (P1), R4.2, R6.2, R8.1
- net DIO10: now also J1.4 (P4); no longer J1.2 (P2), R4.1
- net DIO7: now also J1.2 (P2), R4.2; no longer J1.4 (P4), R6.1
- net GND: now also C12.1, C13.1, C14.1, C4.2, C5.2, C6.2, R13.1, U1.33 (GND), C20.1, C21.1, C22.1, C23.1, C24.1, U2.1 (GND); no longer C4.1, C5.1, C6.1, R13.2
- net at C1.1, C2.1, C3.1: now also R7.2, U1.28 (VDD1V2); no longer R7.1
- net at C12.2, U1.23 (SXTAL0), Y1.1: now also R16.1
- net at C14.2, U1.18 (FXTAL0), Y2.3: now also R6.1
- net DIO12_BUTTON: now reaches U1.30 (DIO12)
- net at TP1.1: now also R7.1; no longer R7.2
- net at TP2.1: now also R8.1; no longer R8.2
- net ANATEST1: no longer names the net of U1.14 (ANATEST1)
- net DIO3 renamed DIO3_LED
- net RESET: no longer names the net of U1.25 (RESETN)
- net RESET: now also R13.2; no longer R13.1
- new net: C20.2, J1.1 (P1), U2.3 (VIN)
- new net: R6.2, TP7.1
- new net: R16.2, TP8.1
Other:
- note added: "*NOTE: Resistors for testing different boot configs. \n -> Omit until needed. *"
- note added: "5/21/2017"
- note added: "Button, rev 2.0"
- note removed: "3/14/2017"
- note removed: "Button, MK.II; rev. 1.2"
- moved on the sheet: C1, C2, C3, C4, C5, C6, C7, C8, C9, J1, R1, R10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

Commit message: rev3 prog
Parts:
- R1, R13, R2, R3, R5: footprint Resistors_SMD:R_0603 -> Resistors_SMD:R_0402
- R4: footprint Resistors_SMD:R_0805 -> Resistors_SMD:R_0402
Connections:
- net DIO2_LED: now reaches U1.10 (DIO2)
- net DIO3_LED: no longer names the net of U1.9 (DIO3)
Changed lines of the file:
@@
 F 0 "R13" V 7150 3950 50  0000 C CNN
 F 1 "100k" V 7250 3950 50  0000 C CNN
-F 2 "Resistors_SMD:R_0603" V 7180 3950 50  0001 C CNN
+F 2 "Resistors_SMD:R_0402" V 7180 3950 50  0001 C CNN
 F 3 "" H 7250 3950 50  0001 C CNN
 	1    7250 3950
@@
 F 0 "R3" H 2100 1950 50  0000 C CNN
 F 1 "100k" V 2000 1800 50  0000 C CNN
-F 2 "Resistors_SMD:R_0603" V 1930 1800 50  0001 C CNN
+F 2 "Resistors_SMD:R_0402" V 1930 1800 50  0001 C CNN
 F 3 "" H 2000 1800 50  0001 C CNN
 	1    2000 1800
@@
 NoConn ~ 5200 5350
 NoConn ~ 5200 5250
-NoConn ~ 5200 5150
 NoConn ~ 5200 4950
 NoConn ~ 5200 4850
@@
 F 0 "R4" H 2750 1800 50  0000 C CNN
 F 1 "100k" V 2600 1800 50  0000 C CNN
-F 2 "Resistors_SMD:R_0805" V 2530 1800 50  0001 C CNN
+F 2 "Resistors_SMD:R_0402" V 2530 1800 50  0001 C CNN
 F 3 "" H 2600 1800 50  0001 C CNN
 	1    2600 1800
@@
 F 0 "R2" H 1850 1950 50  0000 C CNN
 F 1 "100k" V 1750 1800 50  0000 C CNN
-F 2 "Resistors_SMD:R_0603" V 1680 1800 50  0001 C CNN
+F 2 "Resistors_SMD:R_0402" V 1680 1800 50  0001 C CNN
 F 3 "" H 1750 1800 50  0001 C CNN
 	1    1750 1800
@@
 F 0 "R1" H 1600 1950 50  0000 C CNN
 F 1 "100k" V 1500 1800 50  0000 C CNN
-F 2 "Resistors_SMD:R_0603" V 1430 1800 50  0001 C CNN
+F 2 "Resistors_SMD:R_0402" V 1430 1800 50  0001 C CNN
 F 3 "" H 1500 1800 50  0001 C CNN
 	1    1500 1800
@@
 F 0 "R5" H 2150 1650 50  0000 C CNN
 F 1 "100k" V 2250 1800 50  0000 C CNN
-F 2 "Resistors_SMD:R_0603" V 2180 1800 50  0001 C CNN
+F 2 "Resistors_SMD:R_0402" V 2180 1800 50  0001 C CNN
 F 3 "" H 2250 1800 50  0001 C CNN
 	1    2250 1800
@@
 DIO12_BUTTON
 NoConn ~ 5200 3850
-Wire Wire Line
-	5200 5050 5150 5050
-Text HLabel 5150 5050 0    20   Output ~ 0
-DIO3_LED
+Text HLabel 5150 5150 0    20   Output ~ 0
+DIO2_LED
 Text HLabel 12300 6350 0    20   Input ~ 0
-DIO3_LED
+DIO2_LED
 Wire Wire Line
 	5200 4150 5150 4150
@@
 Wire Wire Line
 	3300 5100 3300 4650
+Wire Wire Line
+	5200 5150 5150 5150
+NoConn ~ 5200 5050
 $EndSCHEMATC

Commit message: added folder, button_elder, to button subtree
Parts:
- removed J1: SWD with less, Pin_Headers:Pin_Header_Straight_1x06_Pitch2.54mm, symbol CONN_01X06
- removed R1, R2: 100k, Resistors_SMD:R_0402, symbol R
- added J1: SWD, Pin_Headers:Pin_Header_Straight_1x08_Pitch2.54mm, symbol CONN_01X08
- added J2: RESET_CONN, Pin_Headers:Pin_Header_Straight_1x02_Pitch2.54mm, symbol CONN_01X02
- added J3: ADC_OUT, Pin_Headers:Pin_Header_Straight_1x03_Pitch2.54mm, symbol CONN_01X03
Connections:
- wire segments 119 -> 135
- no-connect marks 11 -> 9
Other:
- moved on the sheet: C20, C21, R13, U2
