File: pcb/kicad/button/button_mkii/peripherals_button.sch (KiCad schematic (older format))
At the start: 8 parts

Commit message: updated design, layout, and appnotes; rev3
Parts:
- removed PB1: pb_basic, Miscellaneous:pb_basic, symbol pb_basic
- added D1: LED (Green-1), LEDs:LED_0402, symbol LED
- added PB1: pb_v2, Buttons_Switches_THT:SW_PUSH-12mm, symbol pb_v2
- added R17: 100k, Resistors_SMD:R_0402, symbol R
- BT1: footprint Batteries:SMD_CoinCell -> Batteries:CoinCell_holder_1060x630
- C18: value CP -> 1uF
- D2: value LED -> LED (Green-2); footprint LEDs:LED_0603 -> LEDs:LED_0402
- R14: value 10k -> 1k
Connections:
- net +3V3: now also C18.1, PB1.1 (ONE); no longer C19.1, R14.1
- net GND: now also D1.1 (K), R17.2; no longer C18.2
- net at BT1.1 (+), D3.2 (A): now also BT1.2 (++), C19.1
- net ANATEST1 renamed LED
- net DIO3: no longer names the net of R14.2
- net DIO3: now also D1.2 (A); no longer C18.1
- new net BUTTON: C18.2, PB1.2 (TWO), R14.1, R17.1
Other:
- note added: "**BATTERY\n + C = dQ/dV\n - Schottky prevents reverse charging into battery"
- note added: "**BUTTON FUNCTIONALITY:\n - When unpressed, button outputs LOW (0V) to uC\n - When pressed, VSRC drives LED; ~1.8V measured\n by uC [limited to ~1mA w/ 1.8V drop across LED]\n - When released, charge drains through pulldown resistor"
- note added: "**LED INDICATOR\n - Requires 1mA, sourced by uC"
- note added: "Not required, current limiter"
- moved on the sheet: BT1, C18, C19, D2, D3, R14, R15
