File: pcb/kicad/button/button_mkii/peripherals_button.sch (KiCad schematic (older format))
At the start: 10 parts

Commit message: rev3.1_layout
Parts:
- removed BT1: Battery, Batteries:batt_holder3035, symbol Battery
- added BT1: Battery_cc3035, Batteries:batt_holder3035, symbol Battery_cc3035
- added C25: 1uF, Capacitors_SMD:C_0603_HandSoldering, symbol CP
- added D4: Power thru Battery, Diodes_SMD:D_0603, symbol D_Schottky
Connections:
- net +3V3: now also D4.1 (K)
- net GND: now also BT1.2 (-), C25.2
- net at C19.1, D3.2 (A): now also BT1.1 (+1)
- new net: BT1.2 (-), C25.1, D4.2 (A)
Changed lines of the file:
@@
 Connection ~ 3950 2800
 $Comp
-L +3.3V #PWR026
+L +3.3V #PWR27
 U 1 1 5901624D
 P 2700 1550
-F 0 "#PWR026" H 2700 1400 50  0001 C CNN
+F 0 "#PWR27" H 2700 1400 50  0001 C CNN
 F 1 "+3.3V" H 2700 1690 50  0000 C CNN
 F 2 "" H 2700 1550 50  0001 C CNN
@@
 $EndComp
 $Comp
-L GND #PWR027
+L GND #PWR28
 U 1 1 5901638D
 P 2700 3200
-F 0 "#PWR027" H 2700 2950 50  0001 C CNN
+F 0 "#PWR28" H 2700 2950 50  0001 C CNN
 F 1 "GND" H 2700 3050 50  0000 C CNN
 F 2 "" H 2700 3200 50  0001 C CNN
@@
 $EndComp
 $Comp
-L GND #PWR028
+L GND #PWR31
 U 1 1 59016561
 P 7650 2250
-F 0 "#PWR028" H 7650 2000 50  0001 C CNN
+F 0 "#PWR31" H 7650 2000 50  0001 C CNN
 F 1 "GND" H 7650 2100 50  0000 C CNN
 F 2 "" H 7650 2250 50  0001 C CNN
@@
 $EndComp
 $Comp
-L GND #PWR029
+L GND #PWR30
 U 1 1 59016756
 P 3950 2850
-F 0 "#PWR029" H 3950 2600 50  0001 C CNN
+F 0 "#PWR30" H 3950 2600 50  0001 C CNN
 F 1 "GND" H 3950 2700 50  0000 C CNN
 F 2 "" H 3950 2850 50  0001 C CNN
@@
 $EndComp
 $Comp
-L +3.3V #PWR030
+L +3.3V #PWR29
 U 1 1 59016919
 P 3950 2000
-F 0 "#PWR030" H 3950 1850 50  0001 C CNN
+F 0 "#PWR29" H 3950 1850 50  0001 C CNN
 F 1 "+3.3V" H 3950 2140 50  0000 C CNN
 F 2 "" H 3950 2000 50  0001 C CNN
@@
 	0    1    1    0
 $EndComp
-Wire Wire Line
-	3950 2800 4450 2800
 $Comp
 L pb_v2 PB1
@@
 $EndComp
 $Comp
-L GND #PWR031
+L GND #PWR26
 U 1 1 5929FDB6
 P 1400 2850
-F 0 "#PWR031" H 1400 2600 50  0001 C CNN
+F 0 "#PWR26" H 1400 2600 50  0001 C CNN
 F 1 "GND" H 1400 2700 50  0000 C CNN
 F 2 "" H 1400 2850 50  0001 C CNN
@@
 Wire Wire Line
 	1400 2800 1400 2850
-$Comp
-L Battery BT1
-U 1 1 59323796
+Connection ~ 3950 2400
+$Comp
+L CP C25
+U 1 1 5933A6A7
+P 4900 2600
+F 0 "C25" H 5050 2650 50  0000 L CNN
+F 1 "1uF" H 5050 2550 50  0000 L CNN
+F 2 "Capacitors_SMD:C_0603_HandSoldering" H 4938 2450 50  0001 C CNN
+F 3 "" H 4900 2600 50  0001 C CNN
+	1    4900 2600
+	1    0    0    -1
+$EndComp
+$Comp
+L D_Schottky D4
+U 1 1 5933A6F4
+P 4900 2200
+F 0 "D4" V 4800 2350 50  0000 C CNN
+F 1 "Power thru Battery" V 4900 2650 50  0000 C CNN
+F 2 "Diodes_SMD:D_0603" H 4900 2200 50  0001 C CNN
+F 3 "" H 4900 2200 50  0001 C CNN
+	1    4900 2200
+	0    1    1    0
+$EndComp
+$Comp
+L Battery_cc3035 BT1
+U 1 1 5933BCAE
 P 4450 2600
 F 0 "BT1" H 4550 2700 50  0000 L CNN
-F 1 "Battery" H 4550 2600 50  0000 L CNN
+F 1 "Battery_cc3035" H 4250 1900 50  0000 L CNN
 F 2 "Batteries:batt_holder3035" V 4450 2660 50  0001 C CNN
 F 3 "" V 4450 2660 50  0001 C CNN
@@
 $EndComp
 Wire Wire Line
-	4450 2400 3950 2400
-Connection ~ 3950 2400
+	3950 2800 4900 2800
+Wire Wire Line
+	4900 2800 4900 2750
+Connection ~ 4450 2800
+Wire Wire Line
+	4900 2450 4900 2350
+Wire Wire Line
+	4500 2400 4900 2400
+Connection ~ 4900 2400
+Wire Wire Line
+	4400 2400 3950 2400
+Wire Wire Line
+	4900 2050 4900 2000
+Wire Wire Line
+	4900 2000 3950 2000
 $EndSCHEMATC
