File: pcb/kicad/button/button_mkii/_saved_button.sch (KiCad schematic (older format))
At the start: 48 parts, among them J1 CONN_01X06, J2 RESET_CONN, J3 CONN_01X05, U1 STBlueNRG-1, U2 TLV1117LV-3V, Y1 Xtal 32.768kHz, Y2 XTAL 32MHz

Commit message: rev3.1
Connections:
- net ADC1: now also J3.3 (P3); no longer J3.2 (P2)
- net ADC2: now also J3.2 (P2); no longer J3.3 (P3)
Changed lines of the file:
@@
 $EndComp
 $Comp
-L GND #PWR01
+L GND #PWR8
 U 1 1 58B79F8B
 P 5100 3100
-F 0 "#PWR01" H 5100 2850 50  0001 C CNN
+F 0 "#PWR8" H 5100 2850 50  0001 C CNN
 F 1 "GND" H 5100 2950 50  0000 C CNN
 F 2 "" H 5100 3100 50  0001 C CNN
@@
 $EndComp
 $Comp
-L GND #PWR02
+L GND #PWR22
 U 1 1 58B7D8A0
 P 9400 4150
-F 0 "#PWR02" H 9400 3900 50  0001 C CNN
+F 0 "#PWR22" H 9400 3900 50  0001 C CNN
 F 1 "GND" H 9400 4000 50  0000 C CNN
 F 2 "" H 9400 4150 50  0001 C CNN
@@
 $EndComp
 $Comp
-L GND #PWR03
+L GND #PWR23
 U 1 1 58B805C2
 P 9550 4950
-F 0 "#PWR03" H 9550 4700 50  0001 C CNN
+F 0 "#PWR23" H 9550 4700 50  0001 C CNN
 F 1 "GND" H 9550 4800 50  0000 C CNN
 F 2 "" H 9550 4950 50  0001 C CNN
@@
 $EndComp
 $Comp
-L GND #PWR04
+L GND #PWR21
 U 1 1 58B8067E
 P 9300 5350
-F 0 "#PWR04" H 9300 5100 50  0001 C CNN
+F 0 "#PWR21" H 9300 5100 50  0001 C CNN
 F 1 "GND" H 9300 5200 50  0000 C CNN
 F 2 "" H 9300 5350 50  0001 C CNN
@@
 $EndComp
 $Comp
-L GND #PWR05
+L GND #PWR19
 U 1 1 58C98635
 P 8350 5150
-F 0 "#PWR05" H 8350 4900 50  0001 C CNN
+F 0 "#PWR19" H 8350 4900 50  0001 C CNN
 F 1 "GND" H 8350 5000 50  0000 C CNN
 F 2 "" H 8350 5150 50  0001 C CNN
@@
 $EndComp
 $Comp
-L GND #PWR06
+L GND #PWR20
 U 1 1 58C986F7
 P 8750 5150
-F 0 "#PWR06" H 8750 4900 50  0001 C CNN
+F 0 "#PWR20" H 8750 4900 50  0001 C CNN
 F 1 "GND" H 8750 5000 50  0000 C CNN
 F 2 "" H 8750 5150 50  0001 C CNN
@@
 $EndComp
 $Comp
-L GND #PWR07
+L GND #PWR10
 U 1 1 58F95B92
 P 6050 5850
-F 0 "#PWR07" H 6050 5600 50  0001 C CNN
+F 0 "#PWR10" H 6050 5600 50  0001 C CNN
 F 1 "GND" H 6050 5700 50  0000 C CNN
 F 2 "" H 6050 5850 50  0001 C CNN
@@
 $EndComp
 $Comp
-L GND #PWR08
+L GND #PWR18
 U 1 1 58F9F433
 P 8000 5600
-F 0 "#PWR08" H 8000 5350 50  0001 C CNN
+F 0 "#PWR18" H 8000 5350 50  0001 C CNN
 F 1 "GND" H 8000 5450 50  0000 C CNN
 F 2 "" H 8000 5600 50  0001 C CNN
@@
 $EndComp
 $Comp
-L GND #PWR09
+L GND #PWR13
 U 1 1 58FA4AD5
 P 7100 3750
-F 0 "#PWR09" H 7100 3500 50  0001 C CNN
+F 0 "#PWR13" H 7100 3500 50  0001 C CNN
 F 1 "GND" H 7100 3800 50  0000 C CNN
 F 2 "" H 7100 3750 50  0001 C CNN
@@
 $EndComp
 $Comp
-L +3.3V #PWR010
+L +3.3V #PWR11
 U 1 1 58FD19CC
 P 6450 2450
-F 0 "#PWR010" H 6450 2300 50  0001 C CNN
+F 0 "#PWR11" H 6450 2300 50  0001 C CNN
 F 1 "+3.3V" H 6450 2590 50  0000 C CNN
 F 2 "" H 6450 2450 50  0001 C CNN
@@
 $EndComp
 $Comp
-L GND #PWR011
+L GND #PWR17
 U 1 1 58FD3CEF
 P 7900 3050
-F 0 "#PWR011" H 7900 2800 50  0001 C CNN
+F 0 "#PWR17" H 7900 2800 50  0001 C CNN
 F 1 "GND" H 7900 2900 50  0000 C CNN
 F 2 "" H 7900 3050 50  0001 C CNN
@@
 $EndComp
 $Comp
-L +3.3V #PWR012
+L +3.3V #PWR14
 U 1 1 58FD8B59
 P 7250 2450
-F 0 "#PWR012" H 7250 2300 50  0001 C CNN
+F 0 "#PWR14" H 7250 2300 50  0001 C CNN
 F 1 "+3.3V" H 7250 2590 50  0000 C CNN
 F 2 "" H 7250 2450 50  0001 C CNN
@@
 DIO9
 $Comp
-L GND #PWR013
+L GND #PWR1
 U 1 1 59031CC6
 P 2000 2000
-F 0 "#PWR013" H 2000 1750 50  0001 C CNN
+F 0 "#PWR1" H 2000 1750 50  0001 C CNN
 F 1 "GND" H 2000 1850 50  0000 C CNN
 F 2 "" H 2000 2000 50  0001 C CNN
@@
 $EndComp
 $Comp
-L +3V3 #PWR014
+L +3V3 #PWR3
 U 1 1 59046761
 P 3300 4100
-F 0 "#PWR014" H 3300 3950 50  0001 C CNN
+F 0 "#PWR3" H 3300 3950 50  0001 C CNN
 F 1 "+3V3" H 3300 4240 50  0000 C CNN
 F 2 "" H 3300 4100 50  0001 C CNN
@@
 $EndComp
 $Comp
-L GND #PWR015
+L GND #PWR4
 U 1 1 59046D5A
 P 3450 4100
-F 0 "#PWR015" H 3450 3850 50  0001 C CNN
+F 0 "#PWR4" H 3450 3850 50  0001 C CNN
 F 1 "GND" H 3450 3950 50  0000 C CNN
 F 2 "" H 3450 4100 50  0001 C CNN
@@
 	1    0    0    -1
 $EndComp
+Text GLabel 4700 5700 1    20   UnSpc ~ 0
+ADC1
 Text GLabel 4800 5700 1    20   UnSpc ~ 0
-ADC1
-Text GLabel 4700 5700 1    20   UnSpc ~ 0
 ADC2
 $Comp
-L +3V3 #PWR016
+L +3V3 #PWR6
 U 1 1 5906178E
 P 4250 4950
-F 0 "#PWR016" H 4250 4800 50  0001 C CNN
+F 0 "#PWR6" H 4250 4800 50  0001 C CNN
 F 1 "+3V3" H 4250 5090 50  0000 C CNN
 F 2 "" H 4250 4950 50  0001 C CNN
@@
 $EndComp
 $Comp
-L GND #PWR017
+L GND #PWR12
 U 1 1 5923B02E
 P 7100 3050
-F 0 "#PWR017" H 7100 2800 50  0001 C CNN
+F 0 "#PWR12" H 7100 2800 50  0001 C CNN
 F 1 "GND" H 7100 2900 50  0000 C CNN
 F 2 "" H 7100 3050 50  0001 C CNN
@@
 $EndComp
 $Comp
-L GND #PWR018
+L GND #PWR9
 U 1 1 592433D3
 P 5750 3050
-F 0 "#PWR018" H 5750 2800 50  0001 C CNN
+F 0 "#PWR9" H 5750 2800 50  0001 C CNN
 F 1 "GND" H 5750 2900 50  0000 C CNN
 F 2 "" H 5750 3050 50  0001 C CNN
@@
 $EndComp
 $Comp
-L GND #PWR019
+L GND #PWR5
 U 1 1 5926C633
 P 3750 5450
-F 0 "#PWR019" H 3750 5200 50  0001 C CNN
+F 0 "#PWR5" H 3750 5200 50  0001 C CNN
 F 1 "GND" H 3750 5300 50  0000 C CNN
 F 2 "" H 3750 5450 50  0001 C CNN
@@
 DIO7
 $Comp
-L +3V3 #PWR020
+L +3V3 #PWR2
 U 1 1 592AABDE
 P 2600 1600
-F 0 "#PWR020" H 2600 1450 50  0001 C CNN
+F 0 "#PWR2" H 2600 1450 50  0001 C CNN
 F 1 "+3V3" H 2600 1740 50  0000 C CNN
 F 2 "" H 2600 1600 50  0001 C CNN
@@
 NoConn ~ 5200 5050
 $Comp
-L GND #PWR021
+L GND #PWR7
 U 1 1 592F3FC9
 P 5000 5700
-F 0 "#PWR021" H 5000 5450 50  0001 C CNN
+F 0 "#PWR7" H 5000 5450 50  0001 C CNN
 F 1 "GND" H 5000 5550 50  0000 C CNN
 F 2 "" H 5000 5700 50  0001 C CNN
@@
 $EndComp
 $Comp
-L +3.3V #PWR022
+L +3.3V #PWR16
 U 1 1 5930CD8C
 P 7700 3850
-F 0 "#PWR022" H 7700 3700 50  0001 C CNN
+F 0 "#PWR16" H 7700 3700 50  0001 C CNN
 F 1 "+3.3V" H 7700 3990 50  0000 C CNN
 F 2 "" H 7700 3850 50  0001 C CNN
@@
 $EndComp
 $Comp
-L GND #PWR023
+L GND #PWR15
 U 1 1 5932E387
 P 7550 3750
-F 0 "#PWR023" H 7550 3500 50  0001 C CNN
+F 0 "#PWR15" H 7550 3500 50  0001 C CNN
 F 1 "GND" H 7550 3600 50  0000 C CNN
 F 2 "" H 7550 3750 50  0001 C CNN
