File: pcb/kicad/button/button_mkii/button.kicad_pcb (KiCad board)
At the start: 2 copper layers, 168 parts, among them J1 SWD with less, U1 STBlueNRG-1, Y1 Xtal 32.768kHz, Y2 XTAL 16MHz

Commit message: updated design, layout, and appnotes; rev3
Parts:
- removed L3: RFC, Miscellaneous:L_0402
- removed the REF** at (127.9, 99.0)
- removed the REF** at (122.2, 108.6)
- removed the REF** at (130.9, 105.6)
- removed the REF** at (124.2, 101.3)
- removed the REF** at (130.9, 106.2)
- removed the REF** at (124.1, 108.4)
- removed the REF** at (113.0, 81.5)
- removed the REF** at (140.2, 101.9)
- removed the REF** at (130.9, 106.9)
- removed the REF** at (143.6, 100.3)
- removed the REF** at (142.5, 100.3)
- removed the REF** at (127.8, 105.6)
- removed the REF** at (128.4, 105.6)
- removed the REF** at (130.9, 107.5)
- added C20, C21: 1uF, Capacitors_SMD:C_0402, F.Cu at (139.2, 64.3)
- added C22: 1uF, Capacitors_SMD:C_0805, F.Cu at (139.2, 64.3)
- added C23: 0.1uF, Capacitors_SMD:C_0603, F.Cu at (139.2, 64.3)
- added C24: 0.01uF, Capacitors_SMD:C_0402, F.Cu at (139.2, 64.3)
- added R16: 1k, Resistors_SMD:R_0402, F.Cu at (139.2, 64.3)
- added R17: 100k, Resistors_SMD:R_0402, F.Cu at (139.2, 64.3)
- added TP7: Xtal32MHz, Miscellaneous:Measurement_Point_Round-SMD-tiniest, F.Cu at (139.2, 64.3)
- added TP8: Xtal32kHz, Miscellaneous:Measurement_Point_Round-SMD-tiniest, F.Cu at (139.2, 64.3)
- added U2: TLV1117LV-3V, TO_SOT_Packages_SMD:SOT-223, F.Cu at (114.2, 104.5)
- BT1: footprint Batteries:SMD_CoinCell -> Batteries:CoinCell_holder_1060x630
- C1: value 100pF -> 1uF; footprint Capacitors_SMD:C_0402 -> Capacitors_SMD:C_0805; moved to F.Cu
- C14: value 22pF -> 27pF
- C15: value 18pF -> 33pF
- C18: value CP -> 1uF
- C2: footprint Capacitors_SMD:C_0402 -> Capacitors_SMD:C_0603; moved to F.Cu
- C3: value 2.2pF -> 0.01uF; moved to F.Cu
- C4: value 1000pF -> 0.01uF; footprint Capacitors_SMD:C_0402 -> Capacitors_SMD:C_0805; moved to F.Cu
- C5: value 2.2uF -> 1000pF; footprint Capacitors_SMD:C_0402 -> Capacitors_SMD:C_0603; moved to F.Cu
- C6, R10, R11, R12, R3, R7, R9, TP1, TP3, TP4, TP5, TP6: moved to F.Cu
- C7: value 10pF -> 0.01uF; footprint Capacitors_SMD:C_0402 -> Capacitors_SMD:C_0805; moved to F.Cu
- C8: value 1uF -> 1000pF; footprint Capacitors_SMD:C_0402 -> Capacitors_SMD:C_0603; moved to F.Cu
- C9: value 1000pF -> 10pF; moved to F.Cu
- D1: value Power thru SWD -> LED (Green-1); footprint Diodes_SMD:D_0603 -> LEDs:LED_0402
- D2: value LED -> LED (Green-2); footprint LEDs:LED_0603 -> LEDs:LED_0402
- L2: value RFC -> L; footprint Miscellaneous:L_0402 -> Capacitors_SMD:C_0603_HandSoldering
- PB1: value pb_basic -> pb_v2; footprint Miscellaneous:pb_basic -> Buttons_Switches_THT:SW_PUSH-12mm
- R14: value 10k -> 1k
- R6: value 100k -> 1k; footprint Resistors_SMD:R_0603 -> Resistors_SMD:R_0402; moved to F.Cu
- U1: footprint uCs:STBNRG1 -> STBNRG1
- Y2: value XTAL 16MHz -> XTAL 32MHz
- moved R4 153.4 mm to (139.2, 64.3)
- moved TP2 48.0 mm to (139.2, 64.3)
- moved R8 46.8 mm to (139.2, 64.3), turned to 0 degrees
- moved D1 46.1 mm to (139.2, 64.3), turned to 0 degrees
- moved D2 45.8 mm to (139.2, 64.3)
- moved R15 44.3 mm to (139.2, 64.3)
- moved C5 42.5 mm to (139.2, 64.3), turned to 0 degrees
- moved TP3 42.0 mm to (139.2, 64.3)
- moved C6 41.9 mm to (139.2, 64.3), turned to 0 degrees
- moved R9 41.8 mm to (139.2, 64.3)
- moved C4 41.6 mm to (139.2, 64.3), turned to 0 degrees
- moved C16 41.4 mm to (139.2, 64.3), turned to 0 degrees
- moved R7 41.3 mm to (139.2, 64.3), turned to 0 degrees
- moved R6 41.3 mm to (139.2, 64.3), turned to 0 degrees
- moved C3 41.0 mm to (139.2, 64.3), turned to 0 degrees
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Connections:
- net RF0 renamed /RF0
- net RF1 renamed /RF1
- BT1 pad 2: GND -> Net-(BT1-Pad1)
- C12 pad 1: Net-(C12-Pad1) -> GND
- C13 pad 1: Net-(C12-Pad1) -> GND
- C14 pad 1: Net-(C14-Pad1) -> GND
- C17 pad 2: Net-(BAL1-Pad3) -> GND
- C18 pad 1: DIO3 -> +3V3
- C18 pad 2: GND -> /DIO12_BUTTON
- C19 pad 1: +3V3 -> Net-(BT1-Pad1)
- C4 pad 1: GND -> +3V3
- C4 pad 2: +3V3 -> GND
- C5 pad 1: GND -> +3V3
- C5 pad 2: +3V3 -> GND
- C6 pad 1: GND -> +3V3
- C6 pad 2: +3V3 -> GND
- D1 pad 1: +3V3 -> GND
- D2 pad 2: ANATEST1 -> /DIO3_LED
- J1 pad 1: +3V3 -> Net-(C20-Pad2)
- J1 pad 2: DIO10 -> DIO7
- J1 pad 4: DIO7 -> DIO10
- J1 pad 6: Net-(D1-Pad2) -> +3V3
- L2 pad 1: Net-(C12-Pad1) -> Net-(BAL1-Pad3)
- PB1 pad 1: DIO3 -> +3V3
- PB1 pad 2: GND -> /DIO12_BUTTON
- R13 pad 1: RESET -> GND
- R13 pad 2: GND -> Net-(R13-Pad2)
- R14 pad 1: +3V3 -> /DIO12_BUTTON
- R14 pad 2: DIO3 -> Net-(D1-Pad2)
- R4 pad 1: DIO10 -> +3V3
- R4 pad 2: +3V3 -> DIO7
- R6 pad 1: DIO7 -> Net-(C14-Pad2)
- R6 pad 2: +3V3 -> Net-(R6-Pad2)
- R7 pad 1: Net-(C1-Pad1) -> Net-(R7-Pad1)
- R7 pad 2: Net-(R7-Pad2) -> Net-(C1-Pad1)
- R8 pad 1: +3V3 -> Net-(R8-Pad1)
- R8 pad 2: Net-(R8-Pad2) -> +3V3
- TP1 pad 1: Net-(R7-Pad2) -> Net-(R7-Pad1)
- TP2 pad 1: Net-(R8-Pad2) -> Net-(R8-Pad1)
- U1 pad 14: ANATEST1 -> Net-(U1-Pad14)
- U1 pad 25: RESET -> Net-(R13-Pad2)
- U1 pad 30: Net-(U1-Pad30) -> /DIO12_BUTTON
- U1 pad 9: DIO3 -> /DIO3_LED
Routing:
- net +3V3: track 104.9 -> 1.14 mm, vias 12 -> 0
- net (no net): track 0.00 -> 34.6 mm
- net ANATEST1: track 20.4 -> 0.00 mm
- net DIO10: track 14.2 -> 0.00 mm, vias 1 -> 0
- net Net-(C13-Pad2): track 14.2 -> 0.00 mm
- net DIO9: track 13.3 -> 0.00 mm, vias 1 -> 0
- net DIO7: track 11.4 -> 0.00 mm, vias 1 -> 0
- net Net-(C12-Pad2): track 8.43 -> 0.00 mm
- net Net-(C10-Pad1): track 7.19 -> 0.00 mm, vias 1 -> 0
- net DIO3: track 6.94 -> 0.00 mm
- net Net-(C1-Pad1): track 4.65 -> 0.00 mm, vias 1 -> 0
- net Net-(BT1-Pad1): track 4.63 -> 0.00 mm, vias 1 -> 0
- net RESET: track 3.17 -> 0.00 mm
- net ADC2: track 2.91 -> 0.01 mm
- net Net-(D1-Pad2): track 2.87 -> 0.00 mm
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
Commit message: rev3 prog
Parts:
- C18, R14: moved to F.Cu
- C19, D1, D2, D3, PB1, R11, R12, R13, R16, TP5, TP6, TP8: moved to B.Cu
- R10, R3, R8: footprint Resistors_SMD:R_0603 -> Resistors_SMD:R_0402
- R4: footprint Resistors_SMD:R_0805 -> Resistors_SMD:R_0402
- R5: footprint Resistors_SMD:R_0603 -> Resistors_SMD:R_0402; moved to F.Cu
- moved C5 53.2 mm to (126.9, 116.1)
- moved D2 51.8 mm to (135.2, 116.0)
- moved C4 51.4 mm to (131.0, 115.0)
- moved C6 51.1 mm to (128.0, 114.2)
- moved TP2 50.6 mm to (117.9, 110.2)
- moved R15 50.2 mm to (134.9, 114.3)
- moved TP3 50.0 mm to (131.8, 113.8)
- moved TP7 49.6 mm to (129.0, 112.9)
- moved R8 49.4 mm to (117.9, 109.0), turned to 90 degrees
- moved R9 49.2 mm to (130.8, 112.8), turned to 270 degrees
- moved R6 49.2 mm to (127.5, 112.1)
- moved C22 48.9 mm to (119.4, 109.1), turned to 90 degrees
- moved C20 48.8 mm to (112.3, 105.0), turned to 270 degrees
- moved C21 47.6 mm to (114.7, 105.2), turned to 180 degrees
- moved C23 47.4 mm to (117.9, 106.6), turned to 90 degrees
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Connections:
- D2 pad 2: /DIO3_LED -> /DIO2_LED
- U1 pad 10: Net-(U1-Pad10) -> /DIO2_LED
- U1 pad 9: /DIO3_LED -> Net-(U1-Pad9)
- U2 pad 1: Net-(C20-Pad2) -> GND
- U2 pad 2: GND -> +3V3
- U2 pad 3: +3V3 -> Net-(C20-Pad2)
Routing:
- net +3V3: track 1.14 -> 60.2 mm, vias 0 -> 1
- net (no net): track 34.6 -> 5.02 mm
- net DIO10: track 0.00 -> 15.1 mm
- net DIO9: track 0.00 -> 14.8 mm
- net DIO7: track 0.00 -> 14.1 mm
- net Net-(C13-Pad2): track 0.00 -> 12.5 mm
- net Net-(C12-Pad2): track 0.00 -> 10.1 mm
- net Net-(C20-Pad2): track 0.00 -> 9.86 mm
- net Net-(BT1-Pad1): track 0.00 -> 8.26 mm
- net Net-(C10-Pad1): track 0.00 -> 5.96 mm
- net Net-(C1-Pad1): track 0.00 -> 5.90 mm
- net Net-(L1-Pad1): track 0.00 -> 2.09 mm
- net /DIO2_LED: track 0.00 -> 1.03 mm, vias 0 -> 1
- net Net-(R8-Pad1): track 0.00 -> 0.79 mm
- net /DIO12_BUTTON: track 0.00 -> 0.74 mm, vias 0 -> 1

Commit message: rev3 prog, almost there...
Parts:
- R10, R6, R7, R8, TP2, TP4, TP7: moved to B.Cu
- R13: footprint Resistors_SMD:R_0603 -> Resistors_SMD:R_0402
- moved REF** 21.7 mm to (119.6, 100.2)
- moved REF** 12.4 mm to (127.8, 100.2)
- moved C5 11.4 mm to (129.9, 105.2)
- moved C6 9.05 mm to (127.1, 105.2)
- moved REF** 8.59 mm to (143.1, 100.2)
- moved REF** 7.16 mm to (129.6, 95.9)
- moved REF** 7.14 mm to (132.1, 95.9)
- moved REF** 7.09 mm to (130.9, 95.9)
- moved C12 6.86 mm to (129.6, 97.4)
- moved C13 6.86 mm to (132.1, 97.4)
- moved Y1 6.86 mm to (130.9, 99.7)
- moved TP4 5.88 mm to (127.1, 102.4), turned to 90 degrees
- moved R17 5.29 mm to (135.8, 88.8), turned to 270 degrees
- moved R6 5.03 mm to (127.8, 107.1)
- moved TP7 5.03 mm to (128.3, 107.9)
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Connections:
- U2 pad 4: (no net) -> +3V3
Routing:
- net +3V3: track 60.2 -> 145.4 mm, vias 1 -> 11
- net /DIO12_BUTTON: track 0.74 -> 41.8 mm, vias 1 -> 2
- net Net-(R13-Pad2): track 0.00 -> 12.1 mm, vias 0 -> 1
- net Net-(D1-Pad2): track 0.00 -> 8.86 mm, vias 0 -> 1
- net (no net): track 5.02 -> 0.00 mm
- net Net-(BAL1-Pad3): track 3.29 -> 0.00 mm
- net GND: track 17.3 -> 18.8 mm
- net Net-(R12-Pad1): track 0.00 -> 1.06 mm
- net Net-(R11-Pad2): track 0.00 -> 0.90 mm
- net Net-(R16-Pad2): track 0.00 -> 0.87 mm
- net Net-(R6-Pad2): track 0.00 -> 0.85 mm
- net Net-(R10-Pad2): track 0.00 -> 0.84 mm
- net Net-(C12-Pad2): track 10.1 -> 10.9 mm, vias 0 -> 1
- net Net-(C14-Pad2): track 6.14 -> 6.35 mm, vias 0 -> 1
- net Net-(L1-Pad1): track 2.09 -> 2.11 mm, vias 0 -> 1
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
Commit message: button, rev3
Parts:
- C4, C5, R9, TP1, TP3: moved to B.Cu
- R1, R2: footprint Resistors_SMD:R_0603 -> Resistors_SMD:R_0402
- moved C4 11.5 mm to (127.3, 104.2), turned to 90 degrees
- moved REF** 11.0 mm to (145.4, 99.5)
- moved REF** 10.7 mm to (128.2, 97.2)
- moved REF** 10.3 mm to (132.6, 110.2)
- moved REF** 8.22 mm to (126.3, 99.8)
- moved REF** 7.79 mm to (126.2, 102.3)
- moved TP3 7.73 mm to (132.3, 106.1)
- moved C16 7.12 mm to (130.2, 104.6), turned to 270 degrees
- moved R9 7.08 mm to (131.3, 105.8), turned to 45 degrees
- moved REF** 6.62 mm to (121.9, 107.9)
- moved REF** 5.16 mm to (123.3, 110.7)
- moved REF** 4.83 mm to (135.0, 111.7)
- moved REF** 4.83 mm to (135.0, 112.3)
- moved REF** 4.83 mm to (135.0, 109.1)
- moved REF** 4.83 mm to (135.0, 107.8)
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Routing:
- net +3V3: track 145.4 -> 172.7 mm, vias 11 -> 13
- net /DIO2_LED: track 1.03 -> 17.6 mm, vias 1 -> 3
- net Net-(BAL1-Pad3): track 0.00 -> 5.50 mm
- net DIO10: track 15.1 -> 17.5 mm
- net ADC2: track 0.01 -> 2.13 mm
- net Net-(D2-Pad1): track 0.00 -> 2.07 mm, vias 0 -> 1
- net ADC1: track 0.16 -> 2.19 mm
- net Net-(R7-Pad1): track 0.00 -> 1.05 mm
- net Net-(R9-Pad2): track 0.00 -> 0.98 mm
- net GND: track 18.8 -> 19.6 mm
- net Net-(C1-Pad1): track 5.90 -> 6.30 mm, vias 0 -> 1

Commit message: added folder, button_elder, to button subtree
Parts:
- removed R1, R2: 100k, Resistors_SMD:R_0402
- removed the REF** at (132.1, 96.5)
- removed the REF** at (129.6, 96.5)
- removed the REF** at (135.6, 101.9)
- added J2: RESET_CONN, Pin_Headers:Pin_Header_Straight_1x02_Pitch2.54mm, F.Cu at (126.5, 86.3)
- added J3: ADC_OUT, Pin_Headers:Pin_Header_Straight_1x03_Pitch2.54mm, F.Cu at (120.0, 116.8)
- J1: value SWD with less -> SWD; footprint Pin_Headers:Pin_Header_Straight_1x06_Pitch2.54mm -> Pin_Headers:Pin_Header_Straight_1x08_Pitch2.54mm
- moved J1 5.07 mm to (111.7, 104.1)
- moved TP4 1.55 mm to (128.6, 101.7)
- moved REF** 0.84 mm to (127.0, 102.4)
- moved TP5 0.19 mm to (124.8, 99.1)
- moved REF** 0.08 mm to (126.2, 99.7)
Connections:
- J1 pad 2: DIO7 -> Net-(J1-Pad2)
- J1 pad 3: DIO9 -> Net-(J1-Pad3)
- J1 pad 4: DIO10 -> DIO7
- J1 pad 5: GND -> DIO9
- J1 pad 6: +3V3 -> DIO10
- U1 pad 11: Net-(U1-Pad11) -> Net-(J1-Pad3)
- U1 pad 12: Net-(U1-Pad12) -> Net-(J1-Pad2)
- U2 pad 4: +3V3 -> (no net)
Routing:
- net Net-(J1-Pad3): track 0.00 -> 6.15 mm
- net Net-(C20-Pad2): track 9.86 -> 3.71 mm
- net +3V3: track 172.7 -> 173.6 mm
- net /DIO12_BUTTON: track 41.8 -> 42.4 mm
- net Net-(C10-Pad1): track 5.98 -> 6.63 mm
- net Net-(C1-Pad1): track 6.30 -> 6.90 mm
- net Net-(L1-Pad1): track 2.11 -> 2.67 mm
Other:
- rule pad_to_mask_clearance: 0.2 -> 0.0762

Commit message: rev3.1
Parts:
- added C25: 1uF, Capacitors_SMD:C_0603_HandSoldering, B.Cu at (119.0, 113.7)
- added D4: Power thru Battery, Diodes_SMD:D_0603, B.Cu at (115.5, 113.7)
- added REF**: Via_Stitch_Dia0.356mm_Drill0.254mm, Miscellaneous:Via_Stitch_Dia0.356mm_Drill0.254mm, F.Cu at (117.2, 101.7)
- added REF**: Via_Stitch_Dia0.356mm_Drill0.254mm, Miscellaneous:Via_Stitch_Dia0.356mm_Drill0.254mm, F.Cu at (116.2, 103.1)
- added TP3: VBATT2, Miscellaneous:Measurement_Point_Round-SMD-tiniest, F.Cu at (131.1, 62.9)
- BT1: value Battery_Cell -> Battery; footprint Batteries:CoinCell_holder_1060x630 -> Batteries:batt_holder3035
- J1: value SWD -> CONN_01X06; footprint Pin_Headers:Pin_Header_Straight_1x08_Pitch2.54mm -> Pin_Headers:Pin_Header_Straight_1x06_Pitch2.54mm
- J3: value ADC_OUT -> CONN_01X05; footprint Pin_Headers:Pin_Header_Straight_1x03_Pitch2.54mm -> Pin_Headers:Pin_Header_Straight_1x05_Pitch2.54mm
- moved REF** 30.1 mm to (115.7, 104.8)
- moved J3 12.7 mm to (132.7, 116.0), turned to 270 degrees
- moved R5 10.2 mm to (116.8, 100.8), turned to 45 degrees
- moved R3 7.81 mm to (115.5, 102.1), turned to 225 degrees
- moved R13 5.72 mm to (126.1, 98.3)
- moved C19 5.47 mm to (118.9, 89.1), turned to 0 degrees
- moved D3 2.66 mm to (115.5, 89.1)
- moved J1 1.61 mm to (111.6, 102.5)
- moved BT1 1.50 mm to (121.5, 101.4)
- moved C21 0.59 mm to (114.2, 104.9), turned to 225 degrees
- moved C20 0.45 mm to (111.9, 104.8), turned to 180 degrees
- moved J2 0.25 mm to (126.2, 86.4)
- moved R4 0.22 mm to (114.2, 103.3)
- renumbered TP3 to VBATT2
Connections:
- BT1 pad 2: Net-(BT1-Pad1) -> GND
- J1 pad 2: Net-(J1-Pad2) -> DIO7
- J1 pad 3: Net-(J1-Pad3) -> DIO9
- J1 pad 4: DIO7 -> DIO10
- J1 pad 5: DIO9 -> GND
- J1 pad 6: DIO10 -> +3V3
- J3 pad 2: ADC1 -> ADC2
- J3 pad 3: ADC2 -> ADC1
- R13 pad 1: GND -> +3V3
- U1 pad 11: Net-(J1-Pad3) -> Net-(J3-Pad5)
- U1 pad 12: Net-(J1-Pad2) -> Net-(J3-Pad4)
Routing:
- net +3V3: track 173.6 -> 128.8 mm, vias 13 -> 9
- net GND: track 19.3 -> 40.3 mm, vias 0 -> 1
- net /DIO12_BUTTON: track 42.4 -> 22.4 mm, vias 2 -> 1
- net Net-(J2-Pad1): track 12.3 -> 0.32 mm, vias 1 -> 0
- net Net-(J1-Pad3): track 6.15 -> 0.00 mm
- net Net-(BT1-Pad1): track 8.26 -> 14.2 mm
- net DIO10: track 17.5 -> 12.1 mm
- net /DIO2_LED: track 17.6 -> 12.5 mm
- net Net-(C20-Pad2): track 3.71 -> 5.05 mm
- net DIO9: track 14.8 -> 15.9 mm
- net Net-(R11-Pad2): track 0.90 -> 0.00 mm
- net DIO7: track 14.1 -> 13.5 mm

Commit message: rev3.1_layout
Parts:
- removed TP3: VBATT2, Miscellaneous:Measurement_Point_Round-SMD-tiniest
- BT1: value Battery -> Battery_cc3035; footprint Batteries:batt_holder3035 -> batt_holder3035
- moved REF** 22.3 mm to (122.4, 89.1)
- moved REF** 8.63 mm to (132.8, 107.0)
- moved REF** 8.29 mm to (124.4, 108.9)
- moved REF** 6.75 mm to (115.5, 109.9)
- moved REF** 6.50 mm to (116.9, 111.7)
- moved J3 5.42 mm to (134.8, 121.0)
- moved D4 2.93 mm to (115.7, 116.6)
- moved C25 2.90 mm to (119.1, 116.6)
- moved C19 2.85 mm to (119.1, 91.9)
- moved D3 2.85 mm to (115.7, 91.9)
- moved BT1 2.85 mm to (121.7, 104.3)
- moved J2 2.37 mm to (126.0, 88.7), turned to 180 degrees
- moved C22 1.53 mm to (118.1, 109.8)
- moved REF** 1.03 mm to (124.4, 109.6)
- moved REF** 0.97 mm to (127.8, 99.2)
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Connections:
- BT1 pad 2: GND -> Net-(BT1-Pad2)
- C25 pad 1: Net-(BT1-Pad1) -> Net-(BT1-Pad2)
- D4 pad 2: Net-(BT1-Pad1) -> Net-(BT1-Pad2)
- U2 pad 4: (no net) -> +3V3
Routing:
- net GND: track 40.3 -> 19.3 mm, vias 1 -> 0
- net /DIO12_BUTTON: track 22.4 -> 42.4 mm, vias 1 -> 2
- net Net-(J2-Pad1): track 0.32 -> 15.3 mm, vias 0 -> 2
- net Net-(BT1-Pad2): track 0.00 -> 10.8 mm
- net Net-(J3-Pad5): track 0.00 -> 10.2 mm
- net ADC2: track 2.13 -> 10.7 mm
- net ADC1: track 2.19 -> 9.85 mm
- net Net-(BT1-Pad1): track 14.2 -> 7.10 mm
- net Net-(J3-Pad4): track 0.00 -> 6.96 mm
- net /DIO2_LED: track 12.5 -> 18.3 mm, vias 3 -> 1
- net +3V3: track 128.8 -> 127.6 mm
- net Net-(R11-Pad2): track 0.00 -> 0.90 mm
