File: pcb/kicad/button/button_mkii/button_rf.sch (KiCad schematic (older format))
At the start: 3 parts

Commit message: updated design, layout, and appnotes; rev3
Parts:
- added L2: L, Capacitors_SMD:C_0603_HandSoldering, symbol L
Connections:
- net GND: now also C17.2, L2.2
- net at BAL1.3 (A1), C16.1: now also L2.1; no longer C17.2
Other:
- moved on the sheet: C17
Changed lines of the file:
@@
 $EndDescr
 $Comp
-L GND #PWR020
+L GND #PWR022
 U 1 1 590A169C
 P 6250 2600
-F 0 "#PWR020" H 6250 2350 50  0001 C CNN
+F 0 "#PWR022" H 6250 2350 50  0001 C CNN
 F 1 "GND" H 6250 2450 50  0000 C CNN
 F 2 "" H 6250 2600 50  0001 C CNN
@@
 Wire Wire Line
 	4000 3350 4100 3350
-Wire Wire Line
-	5100 3050 5250 3050
 $Comp
-L GND #PWR021
+L GND #PWR023
 U 1 1 59041AB0
-P 5600 3400
-F 0 "#PWR021" H 5600 3150 50  0001 C CNN
-F 1 "GND" H 5600 3250 50  0000 C CNN
-F 2 "" H 5600 3400 50  0001 C CNN
-F 3 "" H 5600 3400 50  0001 C CNN
-	1    5600 3400
+P 5700 3400
+F 0 "#PWR023" H 5700 3150 50  0001 C CNN
+F 1 "GND" H 5700 3250 50  0000 C CNN
+F 2 "" H 5700 3400 50  0001 C CNN
+F 3 "" H 5700 3400 50  0001 C CNN
+	1    5700 3400
 	1    0    0    -1
 $EndComp
 Wire Wire Line
-	5600 3350 5600 3400
+	5700 3350 5700 3400
 $Comp
 L C C16
@@
 L C C17
 U 1 1 590E3EE4
-P 5400 3050
-F 0 "C17" V 5150 2950 50  0000 L CNN
-F 1 "TBD" V 5250 2950 50  0000 L CNN
-F 2 "Capacitors_SMD:C_0402" H 5438 2900 50  0001 C CNN
-F 3 "" H 5400 3050 50  0001 C CNN
-	1    5400 3050
-	0    1    1    0
+P 5700 3200
+F 0 "C17" V 5450 3100 50  0000 L CNN
+F 1 "TBD" V 5550 3100 50  0000 L CNN
+F 2 "Capacitors_SMD:C_0402" H 5738 3050 50  0001 C CNN
+F 3 "" H 5700 3200 50  0001 C CNN
+	1    5700 3200
+	-1   0    0    1
 $EndComp
 Wire Wire Line
-	5100 3350 5600 3350
+	5100 3350 5700 3350
 Connection ~ 5200 3350
 Connection ~ 5200 3050
 Wire Wire Line
-	6150 3050 5550 3050
-Wire Wire Line
-	6150 2000 6150 3050
+	6150 3050 6150 2000
 Wire Wire Line
 	6150 2000 7200 2000
@@
 Wire Wire Line
 	7200 2500 6250 2500
+Connection ~ 5700 3050
+$Comp
+L L L2
+U 1 1 592770C3
+P 5450 3050
+F 0 "L2" V 5400 3050 50  0000 C CNN
+F 1 "L" V 5525 3050 50  0000 C CNN
+F 2 "Capacitors_SMD:C_0603_HandSoldering" H 5450 3050 50  0001 C CNN
+F 3 "" H 5450 3050 50  0001 C CNN
+	1    5450 3050
+	0    -1   -1   0
+$EndComp
+Wire Wire Line
+	5100 3050 5300 3050
+Wire Wire Line
+	5600 3050 6150 3050
 $EndSCHEMATC
