File: pcb/kicad/button/button_mki/button_1_00.sch (KiCad schematic (older format))
At the start: 79 parts, among them J10 GND_OUT, J1001 IO_SMALL_BRD, J1002 IO_SMALL_OUT, J1003 IO_SMALL_IN, J1004 IO_BOT_BRD, J1005 IO_BOT_OUT, J1006 IO_BOT_IN, J1007 IO_TOP_BRD, J1008 IO_TOP_OUT, J11 PWR_OUT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

Commit message: rev3.1
Parts:
- BT1001: symbol Battery_Cell -> Battery_Cell-RESCUE-button_1_00
Other:
- moved on the sheet: U?
Changed lines of the file:
@@
 LIBS:contrib
 LIBS:valves
-LIBS:misc
-LIBS:uCs
-LIBS:coin_cells
 LIBS:button_1_00-cache
 EELAYER 25 0
@@
 $EndComp
 $Comp
-L Battery_Cell BT1001
+L Battery_Cell-RESCUE-button_1_00 BT1001
 U 1 1 59053AF1
 P 5700 6900
@@
 L STBlueNRG-1 U?
 U 1 1 58F497FB
-P 7000 2850
-F 0 "U?" H 7850 2150 50  0000 C CNN
-F 1 "STBlueNRG-1" H 7050 3100 50  0000 C CNN
-F 2 "MLF/QFN32" H 7700 2000 50  0001 C CIN
-F 3 "" H 7000 2850 50  0001 C CNN
-	1    7000 2850
-	1    0    0    -1
-$EndComp
+P 4150 200
+F 0 "U?" H 5000 -500 50  0000 C CNN
+F 1 "STBlueNRG-1" H 4200 450 50  0000 C CNN
+F 2 "MLF/QFN32" H 4850 -650 50  0001 C CIN
+F 3 "" H 4150 200 50  0001 C CNN
+	1    4150 200
+	1    0    0    -1
+$EndComp
